File: p3-u3-w/SD_DAC.kicad_sch (KiCad schematic)
At the start: 26 parts, among them J3 SJ-3524-SMT, J4 473092651, U2 PCM5102A

Commit message: finished schematics, started routing and layout.
Parts:
- C17, C18, C19, C20, C21, C22, C23, C24, C25, C26, C27, C28, C29: footprint (none) -> Capacitor_SMD:C_0603_1608Metric
- J3: footprint SJ-3524-SMT:CUI_SJ-3524-SMT -> SJ_3524_SMT_TR:CUI_SJ-3524-SMT
- J4: footprint CONN12_47309-2651_MOL -> 473092651:CONN12_47309-2651_MOL
- R10, R11, R12, R13, R14, R5, R6, R7, R8, R9: footprint (none) -> Resistor_SMD:R_0603_1608Metric
Connections:
- net +3.3VA is gone; now on net +3.3V: C18.2, C20.2, C22.2, C23.2, C27.2, C28.2, U2.1 (CPVDD), U2.17 (XSMT), U2.20 (DVDD), U2.8 (AVDD)
- net GNDA is gone; now on net GND: C18.1, C19.2, C20.1, C21.2, C22.1, C23.1, C24.1, C25.1, C26.2, C27.1, C28.1, J3.1, U2.19 (DGND), U2.3 (CPGND), U2.9 (AGND)
Other:
- note added: "Star Section"
- note removed: "Need Way of getting GNDA and 3v3A"

Commit message: changed some routing
Parts:
- C17, C18, C19, C20, C21, C22, C23, C24, C25, C26, C27, C28, C29: footprint Capacitor_SMD:C_0603_1608Metric -> Capacitor_SMD:C_0402_1005Metric
- R10, R11, R12, R13, R14, R5, R6, R7, R8, R9: footprint Resistor_SMD:R_0603_1608Metric -> Resistor_SMD:R_0402_1005Metric
Changed lines of the file:
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@@
 			)
 		)
-		(property "Footprint" "Capacitor_SMD:C_0603_1608Metric"
+		(property "Footprint" "Capacitor_SMD:C_0402_1005Metric"
 			(at 98.0948 68.58 0)
 			(effects
@@
 			)
 		)
-		(property "Footprint" "Capacitor_SMD:C_0603_1608Metric"
+		(property "Footprint" "Capacitor_SMD:C_0402_1005Metric"
 			(at 112.0648 113.03 0)
 			(effects
@@
 			)
 		)
-		(property "Footprint" "Capacitor_SMD:C_0603_1608Metric"
+		(property "Footprint" "Capacitor_SMD:C_0402_1005Metric"
 			(at 113.3348 77.47 0)
 			(effects
@@
 			)
 		)
-		(property "Footprint" "Resistor_SMD:R_0603_1608Metric"
+		(property "Footprint" "Resistor_SMD:R_0402_1005Metric"
 			(at 36.83 98.298 90)
 			(effects
@@
 			)
 		)
-		(property "Footprint" "Capacitor_SMD:C_0603_1608Metric"
+		(property "Footprint" "Capacitor_SMD:C_0402_1005Metric"
 			(at 119.6848 77.47 0)
 			(effects
@@
 			)
 		)
-		(property "Footprint" "Resistor_SMD:R_0603_1608Metric"
+		(property "Footprint" "Resistor_SMD:R_0402_1005Metric"
 			(at 111.76 95.758 90)
 			(effects
@@
 			)
 		)
-		(property "Footprint" "Capacitor_SMD:C_0603_1608Metric"
+		(property "Footprint" "Capacitor_SMD:C_0402_1005Metric"
 			(at 61.9252 68.58 0)
 			(effects
@@
 			)
 		)
-		(property "Footprint" "Capacitor_SMD:C_0603_1608Metric"
+		(property "Footprint" "Capacitor_SMD:C_0402_1005Metric"
 			(at 192.0748 45.72 0)
 			(effects
@@
 			)
 		)
-		(property "Footprint" "Resistor_SMD:R_0603_1608Metric"
+		(property "Footprint" "Resistor_SMD:R_0402_1005Metric"
 			(at 100.33 93.218 90)
 			(effects
@@
 			)
 		)
-		(property "Footprint" "Capacitor_SMD:C_0603_1608Metric"
+		(property "Footprint" "Capacitor_SMD:C_0402_1005Metric"
 			(at 104.4448 113.03 0)
 			(effects
@@
 			)
 		)
-		(property "Footprint" "Capacitor_SMD:C_0603_1608Metric"
+		(property "Footprint" "Capacitor_SMD:C_0402_1005Metric"
 			(at 94.2848 123.19 0)
 			(effects
@@
 			)
 		)
-		(property "Footprint" "Capacitor_SMD:C_0603_1608Metric"
+		(property "Footprint" "Capacitor_SMD:C_0402_1005Metric"
 			(at 96.8248 106.68 0)
 			(effects
@@
 			)
 		)
-		(property "Footprint" "Capacitor_SMD:C_0603_1608Metric"
+		(property "Footprint" "Capacitor_SMD:C_0402_1005Metric"
 			(at 41.6052 67.31 0)
 			(effects
@@
 			)
 		)
-		(property "Footprint" "Resistor_SMD:R_0603_1608Metric"
+		(property "Footprint" "Resistor_SMD:R_0402_1005Metric"
 			(at 46.99 95.758 90)
 			(effects
@@
 			)
 		)
-		(property "Footprint" "Capacitor_SMD:C_0603_1608Metric"
+		(property "Footprint" "Capacitor_SMD:C_0402_1005Metric"
 			(at 33.9852 67.31 0)
 			(effects
@@
 			)
 		)
-		(property "Footprint" "Resistor_SMD:R_0603_1608Metric"
+		(property "Footprint" "Resistor_SMD:R_0402_1005Metric"
 			(at 203.708 59.69 90)
 			(effects
@@
 			)
 		)
-		(property "Footprint" "Resistor_SMD:R_0603_1608Metric"
+		(property "Footprint" "Resistor_SMD:R_0402_1005Metric"
 			(at 46.99 100.838 90)
 			(effects
@@
 			)
 		)
-		(property "Footprint" "Resistor_SMD:R_0603_1608Metric"
+		(property "Footprint" "Resistor_SMD:R_0402_1005Metric"
 			(at 211.328 59.69 90)
 			(effects
@@
 			)
 		)
-		(property "Footprint" "Resistor_SMD:R_0603_1608Metric"
+		(property "Footprint" "Resistor_SMD:R_0402_1005Metric"
 			(at 36.83 93.218 90)
 			(effects
@@
 			)
 		)
-		(property "Footprint" "Capacitor_SMD:C_0603_1608Metric"
+		(property "Footprint" "Capacitor_SMD:C_0402_1005Metric"
 			(at 69.5452 68.58 0)
 			(effects
@@
 			)
 		)
-		(property "Footprint" "Resistor_SMD:R_0603_1608Metric"
+		(property "Footprint" "Resistor_SMD:R_0402_1005Metric"
 			(at 197.358 34.29 90)
 			(effects
@@
 			)
 		)
-		(property "Footprint" "Resistor_SMD:R_0603_1608Metric"
+		(property "Footprint" "Resistor_SMD:R_0402_1005Metric"
 			(at 212.09 38.608 90)
 			(effects
@@
 			)
 		)
-		(property "Footprint" "Capacitor_SMD:C_0603_1608Metric"
+		(property "Footprint" "Capacitor_SMD:C_0402_1005Metric"
 			(at 90.4748 68.58 0)
 			(effects

Commit message: added in some more routing.
Connections:
- net +3.3V: no longer C18.2, C20.2, C22.2, C23.2, C27.2, C28.2, U2.1 (CPVDD), U2.17 (XSMT), U2.20 (DVDD), U2.8 (AVDD)
- net GND: no longer C18.1, C19.2, C20.1, C21.2, C22.1, C23.1, C24.1, C25.1, C26.2, C27.1, C28.1, J3.1, U2.19 (DGND), U2.3 (CPGND), U2.9 (AGND)
- new net +3.3VA: C18.2, C20.2, C22.2, C23.2, C27.2, C28.2, U2.1 (CPVDD), U2.17 (XSMT), U2.20 (DVDD), U2.8 (AVDD)
- new net GNDA: C18.1, C19.2, C20.1, C21.2, C22.1, C23.1, C24.1, C25.1, C26.2, C27.1, C28.1, J3.1, U2.19 (DGND), U2.3 (CPGND), U2.9 (AGND)
Changed lines of the file:
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@@
-	(wire
-		(pts
-			(xy 198.12 114.3) (xy 214.63 114.3)
-		)
-		(stroke
-			(width 0)
-			(type default)
-		)
-	)
 	(wire
 		(pts
@@
 		)
 		(stroke
-			(width 0)
-			(type default)
-		)
-	)
-	(wire
-		(pts
-			(xy 198.12 106.68) (xy 214.63 106.68)
-		)
-		(stroke

Commit message: finished routing need to pass drc
Connections:
- net +3.3VA is gone; now on net +3.3V: C18.2, C20.2, C22.2, C23.2, C27.2, C28.2, U2.1 (CPVDD), U2.17 (XSMT), U2.20 (DVDD), U2.8 (AVDD)
- net GNDA is gone; now on net GND: C18.1, C19.2, C20.1, C21.2, C22.1, C23.1, C24.1, C25.1, C26.2, C27.1, C28.1, J3.1, U2.19 (DGND), U2.3 (CPGND), U2.9 (AGND)
Changed lines of the file:
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@@
+	(wire
+		(pts
+			(xy 198.12 106.68) (xy 214.63 106.68)
+		)
+		(stroke
+			(width 0)
+			(type default)
+		)
+	)
 	(wire
 		(pts
@@
 		)
 		(stroke
+			(width 0)
+			(type default)
+		)
+	)
+	(wire
+		(pts
+			(xy 198.12 114.3) (xy 214.63 114.3)
+		)
+		(stroke
