File: p3-u3-w/p3-u3-w.kicad_pcb (KiCad board)
At the start: 6 copper layers, 14 x 90 mm, 104 parts, among them J1 SWD_pin, J2 Display, J3 SJ-3524-SMT, J4 473092651, J5 UART, J6 12401826E412A, J7 Bat Conn, J8 CONMHF1-SMD-G-T, SW1 SW_SPST, SW2 SW_SPST, SW3 SW_SPST, SW4 SW_SPST, SW5 SW_SPST, SW6 SW_SPST, SW7 SW_SPST, U1 LSM6DSM, U2 PCM5102A, U3 STM32WB55CEUx, U4 LD39050PU33R, U5 TPS63802DLAR, U6 MCP73831T-2ACI/OT, U7 DLF162500LT-5028A1, X1 NX2016SA-32MHZ-EXS00A-CS06654, Y2 32k768

Commit message: made changes acording to angus.
Routing:
- net GND: track 165.4 -> 164.7 mm
- net IMU_INT1: vias 3 -> 2

Commit message: finished the pcb, added in BOM
Parts:
- removed J5: UART, Connector_PinHeader_1.00mm:PinHeader_1x02_P1.00mm_Vertical
- moved C42 3.37 mm to (152.0, 103.0), turned to 180 degrees
- moved L2 2.81 mm to (152.5, 101.0)
- moved C41 2.59 mm to (152.0, 99.0), turned to 180 degrees
- moved U7 2.00 mm to (152.5, 104.6), turned to -90 degrees
- moved J8 0.70 mm to (149.5, 107.0), turned to 90 degrees
Connections:
- U3 pad 11: UART_TX -> unconnected-(U3-PA2-Pad11)
- U3 pad 12: UART_RX -> unconnected-(U3-PA3-Pad12)
Routing:
- net GND: track 164.7 -> 153.2 mm, vias 57 -> 108
- net USB_D-: track 51.5 -> 47.4 mm, vias 5 -> 4
- net +3.3V: track 124.5 -> 127.3 mm, vias 31 -> 32
- net USB_D+: track 43.6 -> 41.3 mm, vias 3 -> 2
- net UART_RX: track 1.79 -> 0.00 mm
- net UART_TX: track 1.58 -> 0.00 mm
- net Net-(J8-SIGNAL): track 1.78 -> 2.40 mm
